File: nfc-business-card.kicad_sch (KiCad schematic)
At the start: 8 parts, among them U1 NT3H2111W0FHKH

Commit message: feat(design): Baskerville/Helvetica typography, larger type scale, centered QR block
- Font registry scripts/fonts.py: single source of truth (face -> TTF/TTC
  with index) shared by preview, KiCad bake, and layout checks
- ENIG name: Georgia Bold -> Baskerville SemiBold (cap 5.2 -> 5.5 mm)
- Silk: Arial -> Helvetica Neue (roles 1.6 -> 1.8 mm, contacts 1.5 -> 1.7 mm)
- QR + contacts block moved down (center 28.5 -> 33.0 mm): roles->QR gap
  0.05 -> 4.55 mm, left column now centered vs antenna zone
- Regenerated assets, PCB, and preview; all layout checks pass
Parts:
- C1: LCSC Part # C158992 -> C301961
Changed lines of the file:
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@@
 		(property "Value" "DNP" (at 109.22 69.85 0) (effects (font (size 1.27 1.27)) (justify left)))
 		(property "Footprint" "NFC_BusinessCard:C_0402_1005Metric" (at 106.68 68.58 0) (effects (font (size 1.27 1.27)) (hide yes)))
-		(property "LCSC Part #" "C158992" (at 106.68 68.58 0) (effects (font (size 1.27 1.27)) (hide yes)))
+		(property "LCSC Part #" "C301961" (at 106.68 68.58 0) (effects (font (size 1.27 1.27)) (hide yes)))
 		(pin "1")
 		(pin "2")
